Commit message: modified laser scanner

File: robots/youbot_base_only.urdf.xacro (robot description, xacro)
@@ -26,6 +26,12 @@
   <xacro:youbot_base name="base"/>
   <!-- base laser front -->
-  <xacro:hokuyo_urg04_laser name="base_laser_front" parent="base" ros_topic="scan_front" update_rate="10" min_angle="-1.57" max_angle="1.57">
-    <origin xyz="0.3 0 -0.03" rpy="0 0 0"/>
+  <xacro:hokuyo_urg04_laser name="base_laser_front" parent="base" ros_topic="scan" update_rate="20" min_angle="0" max_angle="6.279">
+    <origin xyz="0 0 0.15" rpy="0 0 0"/>
   </xacro:hokuyo_urg04_laser>
+  <!-- base laser rear -->
+<!--
+  <xacro:hokuyo_urg04_laser name="base_laser_rear" parent="base" ros_topic="scan" update_rate="15" min_angle="-1.57" max_angle="1.57">
+    <origin xyz="-0.3 0 -0.03" rpy="0 0 3.14159"/>
+  </xacro:hokuyo_urg04_laser>
+-->
 </robot>

File: urdf/sensors/hokuyo_urg04_laser.gazebo.xacro (robot description, xacro)
@@ -14,6 +14,6 @@
             <scan>
                 <horizontal>
-                    <samples>150</samples>
-                    <resolution>1.0</resolution>
+                    <samples>1000</samples>
+                    <resolution>0.33</resolution>
                     <min_angle>${min_angle}</min_angle>
                     <max_angle>${max_angle}</max_angle>
@@ -22,6 +22,6 @@
             <range>
 				<min>0.05</min>
-				<max>5.6</max>
-				<resolution>0.36</resolution>
+				<max>50.0</max>
+				<resolution>0.2</resolution>
 			</range>
         </ray>

Commit message: added in second sensor to test out sensor merging

File: robots/youbot_base_only.urdf.xacro (robot description, xacro)
@@ -26,12 +26,10 @@
   <xacro:youbot_base name="base"/>
   <!-- base laser front -->
-  <xacro:hokuyo_urg04_laser name="base_laser_front" parent="base" ros_topic="base_scan" update_rate="20" min_angle="0" max_angle="6.279">
-    <origin xyz="0 0 0.15" rpy="0 0 0"/>
+  <xacro:hokuyo_urg04_laser name="base_laser_front" parent="base" ros_topic="scan_fl" update_rate="20" min_angle="-2.35619449019" max_angle="2.35619449019">
+    <origin xyz="0.2 0.2 0.15" rpy="0 0 0.785"/>
   </xacro:hokuyo_urg04_laser>
   <!-- base laser rear -->
-<!--
-  <xacro:hokuyo_urg04_laser name="base_laser_rear" parent="base" ros_topic="scan" update_rate="15" min_angle="-1.57" max_angle="1.57">
-    <origin xyz="-0.3 0 -0.03" rpy="0 0 3.14159"/>
+  <xacro:hokuyo_urg04_laser name="base_laser_rear" parent="base" ros_topic="scan_br" update_rate="20" min_angle="-2.35619449019" max_angle="2.35619449019">
+    <origin xyz="-0.2 -0.2 0.15" rpy="0 0 -2.355796"/>
   </xacro:hokuyo_urg04_laser>
--->
 </robot>

File: urdf/sensors/hokuyo_urg04_laser.gazebo.xacro (robot description, xacro)
@@ -14,6 +14,6 @@
             <scan>
                 <horizontal>
-                    <samples>1000</samples>
-                    <resolution>0.6</resolution>
+                    <samples>720</samples>
+                    <resolution>1.0</resolution>
                     <min_angle>${min_angle}</min_angle>
                     <max_angle>${max_angle}</max_angle>
@@ -23,5 +23,5 @@
 				<min>0.05</min>
 				<max>50.0</max>
-				<resolution>0.4</resolution>
+				<resolution>0.01</resolution>
 			</range>
         </ray>
