Commit message: improved wheel slippage by changing wheel radius to match gazebo radius

File: urdf/youbot_base/base.urdf.xacro (robot description, xacro)
@@ -19,13 +19,16 @@
   <xacro:property name="wheel_offset_z" value="0.0"/>
   <xacro:property name="wheel_mass" value="1.4"/>
-  <xacro:property name="wheel_radius" value="0.0475"/>
+  <!--<xacro:property name="wheel_radius" value="0.0475"/>-->
+  <xacro:property name="wheel_radius" value="0.05"/>
   <xacro:property name="wheel_length" value="0.005"/>
   <xacro:property name="caster_joint_damping" value="1.0"/>
   <xacro:property name="caster_joint_friction" value="1.0"/>
+  <!--<xacro:property name="caster_joint_friction" value="100.0"/>-->
   <xacro:property name="caster_joint_effort" value="30"/>
   <xacro:property name="caster_joint_velocity" value="10"/>
   <xacro:property name="caster_joint_safety_k_velocity" value="10.0"/>
   <xacro:property name="wheel_joint_damping" value="1.0"/>
-  <xacro:property name="wheel_joint_friction" value="1.0"/>
+  <!--<xacro:property name="wheel_joint_friction" value="1.0"/>-->
+    <xacro:property name="wheel_joint_friction" value="1.0"/>
   <xacro:property name="wheel_joint_effort" value="30"/>
   <xacro:property name="wheel_joint_velocity" value="10"/>
